File: testbench.brd (EAGLE design)
At the start: 100 x 50 mm, 100 parts, among them IC1 74LS595D, IC2 74LS595D, Q1 MOSFET-N, Q2 MOSFET-N, Q3 MOSFET-N, Q4 MOSFET-N, Q5 MOSFET-N, Q6 MOSFET-N, U1 ATMEGA328P_TQFP, U2 KA7805ERTF, Y1 20MHz

Commit message: v 1.0 - REV_A
You can find all the gerbers and the BOM. Sent to Fab House.
Parts:
- added F1: PTCSMD-W, SparkFun-PowerIC:PTC-1206-WIDE
- moved U$3 41.4 mm to (83.3, 23.3)
- moved U$1 29.9 mm to (54.8, 46.2), turned to 180 degrees
- moved U$2 25.6 mm to (2.61, 44.2), turned to 180 degrees
Connections:
- new net +24VHE: D1.C, D2.C, D3.C, D4.C, D5.C, D6.C, F1.2, HOTEND1.1, HOTEND2.1, HOTEND3.1, HOTEND4.1, HOTEND5.1, HOTEND6.1, R1.2, R13.2, R17.2, R21.2, R5.2, R9.2
- net +24V: now also F1.1; no longer D1.C, D2.C, D3.C, D4.C, D5.C, D6.C, HOTEND1.1, HOTEND2.1, HOTEND3.1, HOTEND4.1, HOTEND5.1, HOTEND6.1, R1.2, R13.2, R17.2, R21.2, R5.2, R9.2
Routing:
- net +24V: track 21.8 -> 19.8 mm
- added copper zone on layer 1, net +24VHE
Other:
- board text added: "+5V"
- board text added: "DTR"
- board text added: "Hotend TestBench Marc Cobler - June 2015 BCN3D Technologies Fundacio CIM ___________________ v 1.0 - REV_A"
- board text added: "NC"
- board text added: "RX"
- board text added: "TX"
- board text removed: "Hotend TestBench Marc Cobler - Spring 2015 BCN3D Technologies Fundacio CIM"

Commit message: All the code for the Hotend Test Jig!
Updated BOM
All the code, untested yet
Updated crystal frequency
Parts:
- Y1: value 20MHz -> 16MHz
Changed lines of the file:
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@@
 <attribute name="MPN" value="ATMEGA328-AU" x="30.9372" y="36.5252" size="1.778" layer="27" display="off"/>
 </element>
-<element name="Y1" library="SparkFun-FreqCtrl" package="HC49US" value="20MHz" x="19.3802" y="31.5214" smashed="yes" rot="R180">
+<element name="Y1" library="SparkFun-FreqCtrl" package="HC49US" value="16MHz" x="19.3802" y="31.5214" smashed="yes" rot="R180">
 <attribute name="NAME" x="16.0782" y="34.163" size="0.8128" layer="25" ratio="10"/>
 <attribute name="OC_FARNELL" value="1842224" x="19.3802" y="31.5214" size="1.778" layer="27" rot="R180" display="off"/>
